File: corbit.kicad_sch (KiCad schematic)
At the start: 0 parts

Commit message: Initial commit
Parts:
- added D1, D10, D11, D12, D13, D14, D15, D16, D17, D18, D19, D2, D20, D21, D3, D4, D5, D6, D7, D8, D9: D, symbol Device:D
- added J1: Conn_01x02, symbol Connector_Generic:Conn_01x02
- added SW1, SW10, SW11, SW12, SW13, SW14, SW15, SW16, SW17, SW18, SW19, SW2, SW20, SW21, SW3, SW4, SW5, SW6, SW7, SW8, SW9: SW_Push, symbol Switch:SW_Push
- added SW22: SW_SPDT, symbol Switch:SW_SPDT
- added U1: XIAO-nRF52840-Plus-SMD, Seeed_Studio_XIAO_Series:XIAO-nRF52840-Plus-SMD, symbol SeedStudio:XIAO-nRF52840_Plus_SMD
Connections:
- new net: J1.1 (Pin_1), SW22.2 (B)
- new net: D5.2 (A), SW5.2
- new net: D19.2 (A), SW19.2
- new net: D20.2 (A), SW20.2
- new net: D11.2 (A), SW11.2
- new net: D15.2 (A), SW15.2
- new net: D6.2 (A), SW6.2
- new net: D3.2 (A), SW3.2
- new net: D21.2 (A), SW21.2
- new net: D10.2 (A), SW10.2
- new net: D4.2 (A), SW4.2
- new net: D13.2 (A), SW13.2
- new net: D9.2 (A), SW9.2
- new net: D12.2 (A), SW12.2
- new net: D8.2 (A), SW8.2
- new net: D16.2 (A), SW16.2
- new net: D7.2 (A), SW7.2
- new net: D14.2 (A), SW14.2
- new net: D18.2 (A), SW18.2
- new net: D1.2 (A), SW1.2
- new net: D17.2 (A), SW17.2
- new net: D2.2 (A), SW2.2
- new net Col0: SW1.1, SW15.1, SW8.1, U1.4 (P0.29_A3_D3)
- new net Col1: SW16.1, SW2.1, SW9.1, U1.5 (P0.04_A4_D4_SDA)
- new net Col2: SW10.1, SW17.1, SW3.1, U1.6 (P0.05_A5_D5_SCL)
- new net Col3: SW11.1, SW18.1, SW4.1, U1.7 (P1.11_D6_TX)
- new net Col4: SW12.1, SW19.1, SW5.1, U1.10 (P1.14_D9_MISO)
- new net Col5: SW13.1, SW20.1, SW6.1, U1.9 (P1.13_D8_SCK)
- new net Col6: SW14.1, SW21.1, SW7.1, U1.8 (P1.12_D7_RX)
- new net GND: J1.2 (Pin_2), U1.13 (GND), U1.27 (GND), U1.33 (GND)
- new net Row0: D1.1 (K), D2.1 (K), D3.1 (K), D4.1 (K), D5.1 (K), D6.1 (K), D7.1 (K), U1.1 (P0.02_A0_D0)
- new net Row1: D10.1 (K), D11.1 (K), D12.1 (K), D13.1 (K), D14.1 (K), D8.1 (K), D9.1 (K), U1.2 (P0.03_A1_D1)
- new net Row2: D15.1 (K), D16.1 (K), D17.1 (K), D18.1 (K), D19.1 (K), D20.1 (K), D21.1 (K), U1.3 (P0.28_A2_D2)
- new net VBAT_SW: SW22.3 (C), U1.32 (VBAT)
- no-connect marks 0 -> 1

Commit message: fix sch
Connections:
- no-connect marks 1 -> 16
