File: corbit.kicad_pcb (KiCad board)
At the start: 2 copper layers, 147 x 94 mm, 44 parts, among them J1 Conn_01x02, SW1 SW_Push, SW10 SW_Push, SW11 SW_Push, SW12 SW_Push, SW13 SW_Push, SW14 SW_Push, SW15 SW_Push, SW16 SW_Push, SW17 SW_Push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

Commit message: fixed direction of diode and slide switch
Parts:
- D1, D10, D11, D12, D13, D14, D15, D16, D17, D18, D19, D2, D20, D3, D4, D5, D6, D7, D8, D9, J1, SW22: moved to B.Cu
- moved J1 3.00 mm to (178.4, 96.0), turned to 90 degrees
- moved D20 1.00 mm to (176.0, 128.0)
- moved SW21 0.99 mm to (191.3, 130.1)
- moved SW22 0.60 mm to (181.0, 104.0), turned to -90 degrees
