File: reel.kicad_pcb (KiCad board)
At the start: 2 copper layers, 144 x 92 mm, 44 parts, among them J1 Conn_01x02, SW1 SW_Push, SW10 SW_Push, SW11 SW_Push, SW12 SW_Push, SW13 SW_Push, SW14 SW_Push, SW15 SW_Push, SW16 SW_Push, SW17 SW_Push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

Commit message: edit
Parts:
- SW1, SW10, SW11, SW12, SW13, SW14, SW15, SW16, SW17, SW18, SW19, SW2, SW20, SW3, SW4, SW5, SW6, SW7, SW8, SW9: footprint corbit:SW_Hotswap_Kailh_Choc_V1_1.00u-NoClickHole -> reel:SW_Hotswap_Kailh_Choc_V1_1.00u-NoClickHole
- SW21: footprint corbit:rotary_encoder_EC05E_Vert -> reel:rotary_encoder_EC05E_Vert
- U1: footprint corbit:XIAO_nRF52840_plus_mki -> reel:XIAO_nRF52840_plus_mki
- moved SW22 1.12 mm to (180.5, 105.0)
