File: reel.kicad_sch (KiCad schematic)
At the start: 44 parts, among them J1 Conn_01x02, SW1 SW_Push, SW10 SW_Push, SW11 SW_Push, SW12 SW_Push, SW13 SW_Push, SW14 SW_Push, SW15 SW_Push, SW16 SW_Push, SW17 SW_Push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

Commit message: rename to ReeL
Parts:
- U1: footprint corbit:XIAO_nRF52840_plus_mki -> reel:XIAO_nRF52840_plus_mki
Changed lines of the file:
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@@
 		)
 		(instances
-			(project "corbit"
+			(project "reel"
 				(path "/46fee64b-d8d5-4529-99df-0fd09c2b7c9b"
 					(reference "#FLG01")
@@
 		)
 		(instances
-			(project "corbit"
+			(project "reel"
 				(path "/46fee64b-d8d5-4529-99df-0fd09c2b7c9b"
 					(reference "J1")
@@
 		)
 		(instances
-			(project "corbit"
+			(project "reel"
 				(path "/46fee64b-d8d5-4529-99df-0fd09c2b7c9b"
 					(reference "D5")
@@
 		)
 		(instances
-			(project "corbit"
+			(project "reel"
 				(path "/46fee64b-d8d5-4529-99df-0fd09c2b7c9b"
 					(reference "D19")
@@
 		)
 		(instances
-			(project "corbit"
+			(project "reel"
 				(path "/46fee64b-d8d5-4529-99df-0fd09c2b7c9b"
 					(reference "#FLG02")
@@
 		)
 		(instances
-			(project "corbit"
+			(project "reel"
 				(path "/46fee64b-d8d5-4529-99df-0fd09c2b7c9b"
 					(reference "D20")
@@
 		)
 		(instances
-			(project "corbit"
+			(project "reel"
 				(path "/46fee64b-d8d5-4529-99df-0fd09c2b7c9b"
 					(reference "D11")
@@
 		)
 		(instances
-			(project "corbit"
+			(project "reel"
 				(path "/46fee64b-d8d5-4529-99df-0fd09c2b7c9b"
 					(reference "SW15")
@@
 		)
 		(instances
-			(project "corbit"
+			(project "reel"
 				(path "/46fee64b-d8d5-4529-99df-0fd09c2b7c9b"
 					(reference "SW6")
@@
 			)
 		)
-		(property "Footprint" "corbit:XIAO_nRF52840_plus_mki"
+		(property "Footprint" "reel:XIAO_nRF52840_plus_mki"
 			(at 60.452 15.494 0)
 			(hide yes)
@@
 		)
 		(instances
-			(project "corbit"
+			(project "reel"
 				(path "/46fee64b-d8d5-4529-99df-0fd09c2b7c9b"
 					(reference "U1")
@@
 		)
 		(instances
-			(project "corbit"
+			(project "reel"
 				(path "/46fee64b-d8d5-4529-99df-0fd09c2b7c9b"
 					(reference "SW3")
@@
 		)
 		(instances
-			(project "corbit"
+			(project "reel"
 				(path "/46fee64b-d8d5-4529-99df-0fd09c2b7c9b"
 					(reference "D15")
@@
 		)
 		(instances
-			(project "corbit"
+			(project "reel"
 				(path "/46fee64b-d8d5-4529-99df-0fd09c2b7c9b"
 					(reference "D10")
@@
 		)
 		(instances
-			(project "corbit"
+			(project "reel"
 				(path "/46fee64b-d8d5-4529-99df-0fd09c2b7c9b"
 					(reference "SW4")
@@
 		)
 		(instances
-			(project "corbit"
+			(project "reel"
 				(path "/46fee64b-d8d5-4529-99df-0fd09c2b7c9b"
 					(reference "D13")
@@
 		)
 		(instances
-			(project "corbit"
+			(project "reel"
 				(path "/46fee64b-d8d5-4529-99df-0fd09c2b7c9b"
 					(reference "#PWR03")
@@
 		)
 		(instances
-			(project "corbit"
+			(project "reel"
 				(path "/46fee64b-d8d5-4529-99df-0fd09c2b7c9b"
 					(reference "D9")
@@
 		)
 		(instances
-			(project "corbit"
+			(project "reel"
 				(path "/46fee64b-d8d5-4529-99df-0fd09c2b7c9b"
 					(reference "#PWR05")
@@
 		)
 		(instances
-			(project "corbit"
+			(project "reel"
 				(path "/46fee64b-d8d5-4529-99df-0fd09c2b7c9b"
 					(reference "D12")
@@
 		)
 		(instances
-			(project "corbit"
+			(project "reel"
 				(path "/46fee64b-d8d5-4529-99df-0fd09c2b7c9b"
 					(reference "SW5")
@@
 		)
 		(instances
-			(project "corbit"
+			(project "reel"
 				(path "/46fee64b-d8d5-4529-99df-0fd09c2b7c9b"
 					(reference "D8")
@@
 		)
 		(instances
-			(project "corbit"
+			(project "reel"
 				(path "/46fee64b-d8d5-4529-99df-0fd09c2b7c9b"
 					(reference "D16")
@@
 		)
 		(instances
-			(project "corbit"
+			(project "reel"
 				(path "/46fee64b-d8d5-4529-99df-0fd09c2b7c9b"
 					(reference "SW22")
@@
 		)
 		(instances
-			(project "corbit"
+			(project "reel"
 				(path "/46fee64b-d8d5-4529-99df-0fd09c2b7c9b"
 					(reference "SW20")
@@
 		)
 		(instances
-			(project "corbit"
+			(project "reel"
 				(path "/46fee64b-d8d5-4529-99df-0fd09c2b7c9b"
 					(reference "SW12")
@@
 		)
 		(instances
-			(project "corbit"
+			(project "reel"
 				(path "/46fee64b-d8d5-4529-99df-0fd09c2b7c9b"
 					(reference "SW8")
@@
 		)
 		(instances
-			(project "corbit"
+			(project "reel"
 				(path "/46fee64b-d8d5-4529-99df-0fd09c2b7c9b"
 					(reference "D7")
@@
 		)
 		(instances
-			(project "corbit"
+			(project "reel"
 				(path "/46fee64b-d8d5-4529-99df-0fd09c2b7c9b"
 					(reference "SW16")
@@
 		)
 		(instances
-			(project "corbit"
+			(project "reel"
 				(path "/46fee64b-d8d5-4529-99df-0fd09c2b7c9b"
 					(reference "D14")
@@
 		)
 		(instances
-			(project "corbit"
+			(project "reel"
 				(path "/46fee64b-d8d5-4529-99df-0fd09c2b7c9b"
 					(reference "SW18")
@@
 		)
 		(instances
-			(project "corbit"
+			(project "reel"
 				(path "/46fee64b-d8d5-4529-99df-0fd09c2b7c9b"
 					(reference "D1")
@@
 		)
 		(instances
-			(project "corbit"
+			(project "reel"
 				(path "/46fee64b-d8d5-4529-99df-0fd09c2b7c9b"
 					(reference "SW9")
@@
 		)
 		(instances
-			(project "corbit"
+			(project "reel"
 				(path "/46fee64b-d8d5-4529-99df-0fd09c2b7c9b"
 					(reference "D17")
@@
 		)
 		(instances
-			(project "corbit"
+			(project "reel"
 				(path "/46fee64b-d8d5-4529-99df-0fd09c2b7c9b"
 					(reference "#PWR01")
@@
 		)
 		(instances
-			(project "corbit"
+			(project "reel"
 				(path "/46fee64b-d8d5-4529-99df-0fd09c2b7c9b"
 					(reference "D3")
@@
 		)
 		(instances
-			(project "corbit"
+			(project "reel"
 				(path "/46fee64b-d8d5-4529-99df-0fd09c2b7c9b"
 					(reference "SW1")
@@
 		)
 		(instances
-			(project "corbit"
+			(project "reel"
 				(path "/46fee64b-d8d5-4529-99df-0fd09c2b7c9b"
 					(reference "SW10")
@@
 		)
 		(instances
-			(project "corbit"
+			(project "reel"
 				(path "/46fee64b-d8d5-4529-99df-0fd09c2b7c9b"
 					(reference "SW21")
@@
 		)
 		(instances
-			(project "corbit"
+			(project "reel"
 				(path "/46fee64b-d8d5-4529-99df-0fd09c2b7c9b"
 					(reference "SW14")
@@
 		)
 		(instances
-			(project "corbit"
+			(project "reel"
 				(path "/46fee64b-d8d5-4529-99df-0fd09c2b7c9b"
 					(reference "SW11")
@@
 		)
 		(instances
-			(project "corbit"
+			(project "reel"
 				(path "/46fee64b-d8d5-4529-99df-0fd09c2b7c9b"
 					(reference "SW13")
@@
 		)
 		(instances
-			(project "corbit"
+			(project "reel"
 				(path "/46fee64b-d8d5-4529-99df-0fd09c2b7c9b"
 					(reference "SW17")
@@
 		)
 		(instances
-			(project "corbit"
+			(project "reel"
 				(path "/46fee64b-d8d5-4529-99df-0fd09c2b7c9b"
 					(reference "SW7")
@@
 		)
 		(instances
-			(project "corbit"
+			(project "reel"
 				(path "/46fee64b-d8d5-4529-99df-0fd09c2b7c9b"
 					(reference "D4")
@@
 		)
 		(instances
-			(project "corbit"
+			(project "reel"
 				(path "/46fee64b-d8d5-4529-99df-0fd09c2b7c9b"
 					(reference "#PWR04")
@@
 		)
 		(instances
-			(project "corbit"
+			(project "reel"
 				(path "/46fee64b-d8d5-4529-99df-0fd09c2b7c9b"
 					(reference "D18")
@@
 		)
 		(instances
-			(project "corbit"
+			(project "reel"
 				(path "/46fee64b-d8d5-4529-99df-0fd09c2b7c9b"
 					(reference "D2")
@@
 		)
 		(instances
-			(project "corbit"
+			(project "reel"
 				(path "/46fee64b-d8d5-4529-99df-0fd09c2b7c9b"
 					(reference "#PWR02")
@@
 		)
 		(instances
-			(project "corbit"
+			(project "reel"
 				(path "/46fee64b-d8d5-4529-99df-0fd09c2b7c9b"
 					(reference "SW2")
@@
 		)
 		(instances
-			(project "corbit"
+			(project "reel"
 				(path "/46fee64b-d8d5-4529-99df-0fd09c2b7c9b"
 					(reference "D6")
@@
 		)
 		(instances
-			(project "corbit"
+			(project "reel"
 				(path "/46fee64b-d8d5-4529-99df-0fd09c2b7c9b"
 					(reference "SW19")

Commit message: fix footprint
Parts:
- SW1, SW10, SW11, SW12, SW13, SW14, SW15, SW16, SW17, SW18, SW19, SW2, SW20, SW3, SW4, SW5, SW6, SW7, SW8, SW9: footprint corbit:SW_Hotswap_Kailh_Choc_V1_1.00u-NoClickHole -> reel:SW_Hotswap_Kailh_Choc_V1_1.00u-NoClickHole
- SW21: footprint corbit:rotary_encoder_EC05E_Vert -> reel:rotary_encoder_EC05E_Vert
Changed lines of the file:
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@@
 			)
 		)
-		(property "Footprint" "corbit:SW_Hotswap_Kailh_Choc_V1_1.00u-NoClickHole"
+		(property "Footprint" "reel:SW_Hotswap_Kailh_Choc_V1_1.00u-NoClickHole"
 			(at 97.79 133.35 0)
 			(hide yes)
@@
 			)
 		)
-		(property "Footprint" "corbit:SW_Hotswap_Kailh_Choc_V1_1.00u-NoClickHole"
+		(property "Footprint" "reel:SW_Hotswap_Kailh_Choc_V1_1.00u-NoClickHole"
 			(at 36.83 116.84 0)
 			(hide yes)
@@
 			)
 		)
-		(property "Footprint" "corbit:SW_Hotswap_Kailh_Choc_V1_1.00u-NoClickHole"
+		(property "Footprint" "reel:SW_Hotswap_Kailh_Choc_V1_1.00u-NoClickHole"
 			(at 67.31 100.33 0)
 			(hide yes)
@@
 			)
 		)
-		(property "Footprint" "corbit:SW_Hotswap_Kailh_Choc_V1_1.00u-NoClickHole"
+		(property "Footprint" "reel:SW_Hotswap_Kailh_Choc_V1_1.00u-NoClickHole"
 			(at 82.55 100.33 0)
 			(hide yes)
@@
 			)
 		)
-		(property "Footprint" "corbit:SW_Hotswap_Kailh_Choc_V1_1.00u-NoClickHole"
+		(property "Footprint" "reel:SW_Hotswap_Kailh_Choc_V1_1.00u-NoClickHole"
 			(at 97.79 100.33 0)
 			(hide yes)
@@
 			)
 		)
-		(property "Footprint" "corbit:SW_Hotswap_Kailh_Choc_V1_1.00u-NoClickHole"
+		(property "Footprint" "reel:SW_Hotswap_Kailh_Choc_V1_1.00u-NoClickHole"
 			(at 97.79 149.86 0)
 			(hide yes)
@@
 			)
 		)
-		(property "Footprint" "corbit:SW_Hotswap_Kailh_Choc_V1_1.00u-NoClickHole"
+		(property "Footprint" "reel:SW_Hotswap_Kailh_Choc_V1_1.00u-NoClickHole"
 			(at 52.07 133.35 0)
 			(hide yes)
@@
 			)
 		)
-		(property "Footprint" "corbit:SW_Hotswap_Kailh_Choc_V1_1.00u-NoClickHole"
+		(property "Footprint" "reel:SW_Hotswap_Kailh_Choc_V1_1.00u-NoClickHole"
 			(at 67.31 116.84 0)
 			(hide yes)
@@
 			)
 		)
-		(property "Footprint" "corbit:SW_Hotswap_Kailh_Choc_V1_1.00u-NoClickHole"
+		(property "Footprint" "reel:SW_Hotswap_Kailh_Choc_V1_1.00u-NoClickHole"
 			(at 36.83 149.86 0)
 			(hide yes)
@@
 			)
 		)
-		(property "Footprint" "corbit:SW_Hotswap_Kailh_Choc_V1_1.00u-NoClickHole"
+		(property "Footprint" "reel:SW_Hotswap_Kailh_Choc_V1_1.00u-NoClickHole"
 			(at 67.31 149.86 0)
 			(hide yes)
@@
 			)
 		)
-		(property "Footprint" "corbit:SW_Hotswap_Kailh_Choc_V1_1.00u-NoClickHole"
+		(property "Footprint" "reel:SW_Hotswap_Kailh_Choc_V1_1.00u-NoClickHole"
 			(at 82.55 116.84 0)
 			(hide yes)
@@
 			)
 		)
-		(property "Footprint" "corbit:SW_Hotswap_Kailh_Choc_V1_1.00u-NoClickHole"
+		(property "Footprint" "reel:SW_Hotswap_Kailh_Choc_V1_1.00u-NoClickHole"
 			(at 36.83 100.33 0)
 			(hide yes)
@@
 			)
 		)
-		(property "Footprint" "corbit:SW_Hotswap_Kailh_Choc_V1_1.00u-NoClickHole"
+		(property "Footprint" "reel:SW_Hotswap_Kailh_Choc_V1_1.00u-NoClickHole"
 			(at 97.79 116.84 0)
 			(hide yes)
@@
 			)
 		)
-		(property "Footprint" "corbit:rotary_encoder_EC05E_Vert"
+		(property "Footprint" "reel:rotary_encoder_EC05E_Vert"
 			(at 125.73 103.886 0)
 			(hide yes)
@@
 			)
 		)
-		(property "Footprint" "corbit:SW_Hotswap_Kailh_Choc_V1_1.00u-NoClickHole"
+		(property "Footprint" "reel:SW_Hotswap_Kailh_Choc_V1_1.00u-NoClickHole"
 			(at 82.55 133.35 0)
 			(hide yes)
@@
 			)
 		)
-		(property "Footprint" "corbit:SW_Hotswap_Kailh_Choc_V1_1.00u-NoClickHole"
+		(property "Footprint" "reel:SW_Hotswap_Kailh_Choc_V1_1.00u-NoClickHole"
 			(at 36.83 133.35 0)
 			(hide yes)
@@
 			)
 		)
-		(property "Footprint" "corbit:SW_Hotswap_Kailh_Choc_V1_1.00u-NoClickHole"
+		(property "Footprint" "reel:SW_Hotswap_Kailh_Choc_V1_1.00u-NoClickHole"
 			(at 67.31 133.35 0)
 			(hide yes)
@@
 			)
 		)
-		(property "Footprint" "corbit:SW_Hotswap_Kailh_Choc_V1_1.00u-NoClickHole"
+		(property "Footprint" "reel:SW_Hotswap_Kailh_Choc_V1_1.00u-NoClickHole"
 			(at 52.07 149.86 0)
 			(hide yes)
@@
 			)
 		)
-		(property "Footprint" "corbit:SW_Hotswap_Kailh_Choc_V1_1.00u-NoClickHole"
+		(property "Footprint" "reel:SW_Hotswap_Kailh_Choc_V1_1.00u-NoClickHole"
 			(at 52.07 116.84 0)
 			(hide yes)
@@
 			)
 		)
-		(property "Footprint" "corbit:SW_Hotswap_Kailh_Choc_V1_1.00u-NoClickHole"
+		(property "Footprint" "reel:SW_Hotswap_Kailh_Choc_V1_1.00u-NoClickHole"
 			(at 52.07 100.33 0)
 			(hide yes)
@@
 			)
 		)
-		(property "Footprint" "corbit:SW_Hotswap_Kailh_Choc_V1_1.00u-NoClickHole"
+		(property "Footprint" "reel:SW_Hotswap_Kailh_Choc_V1_1.00u-NoClickHole"
 			(at 82.55 149.86 0)
 			(hide yes)
