File: right/reel-right.kicad_pcb (KiCad board)
At the start: 2 copper layers, 134 x 86.9 mm, 42 parts, among them J1 Conn_01x02, SW1 SW_Push, SW10 SW_Push, SW11 SW_Push, SW12 SW_Push, SW13 SW_Push, SW14 SW_Push, SW15 SW_Push, SW16 SW_Push, SW17 SW_Push, SW18 SW_Push, SW19 SW_Push, SW2 SW_Push, SW22 SW_SPDT, SW3 SW_Push, SW4 SW_Push, SW5 SW_Push, SW6 SW_Push, SW7 SW_Push, SW8 SW_Push, SW9 SW_Push, U1 XIAO-nRF52840-Plus-SMD

Commit message: Update XIAO BLE footprints
Parts:
- added Ref**: Val**, reel:m2_Spacer_Hole, F.Cu at (146.5, 55.5)
- added Ref**: Val**, reel:m2_Spacer_Hole, F.Cu at (52.5, 74.5)
- added Ref**: Val**, reel:m2_Spacer_Hole, F.Cu at (55.0, 108.0)
- added Ref**: Val**, reel:m2_Spacer_Hole, F.Cu at (170.0, 108.5)
- U1: value XIAO-nRF52840-Plus-SMD -> ~; footprint reel:XIAO_nRF52840_plus_mki -> reel:XIAO_nRF52840_wBAT_wNFC_1
- moved U1 8.00 mm to (59.0, 49.0)
- moved J1 3.53 mm to (52.0, 80.5)
- moved SW22 2.50 mm to (49.2, 90.5)
Connections:
- U1 pad 15: GND -> Col3
- U1 pad 16: VBAT_SW -> Col4
- U1 pad 20: unconnected-(U1-GPIO_0.09-Pad20) -> VBAT_SW
- U1 pad 21: Col1 -> GND
- U1 pad 6: SCLK -> Col1
- U1 pad 8: Col3 -> nCS
- U1 pad 9: Col4 -> SCLK
Routing:
- net Row3: track 1.56 -> 227.3 mm, vias 1 -> 7
- net GND: track 0.00 -> 162.2 mm
- net Col0: track 52.6 -> 191.8 mm, vias 0 -> 2
- net SDIO: track 0.00 -> 136.3 mm, vias 0 -> 1
- net MOTION: track 0.00 -> 134.9 mm, vias 0 -> 2
- net nCS: track 0.00 -> 115.3 mm
- net SCLK: track 0.00 -> 115.1 mm
- net Col1: track 108.7 -> 223.0 mm
- net Col2: track 89.3 -> 166.1 mm, vias 0 -> 2
- net Col3: track 119.3 -> 157.3 mm
- net VBAT_SW: track 0.00 -> 37.7 mm, vias 0 -> 3
- net 3.3V: track 126.7 -> 152.1 mm
- net Col4: track 34.0 -> 52.5 mm
- net Net-(J1-Pin_1): track 0.00 -> 15.8 mm, vias 0 -> 1
- net Row2: track 141.6 -> 134.6 mm, vias 8 -> 9
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